Commit message: added stl models and updated PD control

File: mara_simple_geometry.urdf (robot description, URDF)
Before this commit: robot mara, 7 links, 6 joints
Links:
- link link1: geometry visual cylinder length=.448 radius=.0687
- link link2: geometry visual cylinder length=.41 radius=.03635
- link link3: geometry visual cylinder length=.1824 radius=.03
- link link4: geometry visual cylinder length=.152 radius=.03
- link link5: geometry visual cylinder length=.0762 radius=.02
- link link6: geometry visual cylinder length=.05 radius=.016
Joints:
- joint joint2: origin xyz=0.2 0.0 0.446 rpy=1.57 0 0 -> xyz=0.2 0.0 0.448 rpy=1.57 0 0
- joint joint4: origin xyz=-0.226 0.0 0.152 rpy=0 0 1.57 -> xyz=-0.23 0 0.152 rpy=0 0 1.57
- joint joint5: origin xyz=0 0.0 0.183 rpy=-3.14 0 1.57 -> xyz=0 0.0 0.152 rpy=-3.14 0 1.57
- joint joint6: origin xyz=0 0.0 0.005 rpy=0 0 3.14 -> xyz=0 0.0 0.05 rpy=0 0 3.14
