Commit message: added urdf file

File: mara.urdf (robot description, URDF)
Before this commit: robot mara, 1 links, 0 joints
Links:
- added link link1; visual cylinder length=.448 radius=.07125
- added link link2; visual cylinder length=.41 radius=.04
- added link link3; visual cylinder length=.152 radius=.03
- added link link4; visual cylinder length=.152 radius=.03
- added link link5; visual cylinder length=.05 radius=.02
- added link link6; visual cylinder length=.05 radius=.016
- link base_link: geometry visual box size=.07125 .07125 0.01
Joints:
- added joint joint1: type continuous, parent base_link, child link1, origin xyz=0 0 0 rpy=0 0 -0.785, axis 0 0 1
- added joint joint2: type continuous, parent link1, child link2, origin xyz=0.2 0.0 0.448 rpy=1.57 0 0, axis 1 0 0
- added joint joint3: type continuous, parent link2, child link3, origin xyz=-0.08 0 0.41 rpy=0 0 0, axis 1 0 0
- added joint joint4: type continuous, parent link3, child link4, origin xyz=0.00 0 0.152 rpy=0 0 0, axis 0 0 1
- added joint joint5: type continuous, parent link4, child link5, origin xyz=0 0.0 0.152 rpy=0 0 0, axis 0 1 0
- added joint joint6: type continuous, parent link5, child link6, origin xyz=0 0.0 0.05 rpy=0 0 0, axis 0 0 1

Commit message: added dual arm support via separate jtas nodes for each arm

File: mara.urdf (robot description, URDF)
Before this commit: robot mara, 7 links, 6 joints
Links:
- removed link link1
- removed link link2
- removed link link3
- removed link link4
- removed link link5
- removed link link6
- added link left_link1; visual mesh filename=package://mara/models/MARA_base.dae scale=0.001 0.001 0.001
- added link left_link2; visual mesh filename=package://mara/models/MARA_arm_1.dae scale=0.001 0.001 0.001
- added link left_link3; visual mesh filename=package://mara/models/MARA_arm_2.dae scale=0.001 0.001 0.001
- added link left_link4; visual mesh filename=package://mara/models/MARA_wrist.dae scale=0.001 0.001 0.001
- added link left_link5; visual cylinder length=.0285 radius=.015
- added link left_link6; visual mesh filename=package://mara/models/MARA_gripper.dae scale=0.01 0.01 0.01
- added link right_link1; visual mesh filename=package://mara/models/MARA_base.dae scale=0.001 0.001 0.001
- added link right_link2; visual mesh filename=package://mara/models/MARA_arm_1.dae scale=0.001 0.001 0.001
- added link right_link3; visual mesh filename=package://mara/models/MARA_arm_2.dae scale=0.001 0.001 0.001
- added link right_link4; visual mesh filename=package://mara/models/MARA_wrist.dae scale=0.001 0.001 0.001
- added link right_link5; visual cylinder length=.0285 radius=.015
- added link right_link6; visual mesh filename=package://mara/models/MARA_gripper.dae scale=0.01 0.01 0.01
- link base_link: geometry visual box size=0.74 1.0 0.4
Joints:
- removed joint joint1
- removed joint joint2
- removed joint joint3
- removed joint joint4
- removed joint joint5
- removed joint joint6
- added joint left_joint1: type continuous, parent base_link, child left_link1, origin xyz=-0.19 0.2 0.206 rpy=0 0 0.785, axis 0 0 1, limit lower=-3.14 upper=3.14 effort=30 velocity=0.6
- added joint left_joint2: type continuous, parent left_link1, child left_link2, origin xyz=0.2 0.0 0.446 rpy=1.57 0 0, axis 1 0 0, limit lower=-3.14 upper=3.14 effort=30 velocity=0.6
- added joint left_joint3: type continuous, parent left_link2, child left_link3, origin xyz=-0.08 0 0.41 rpy=3.14 0 0, axis 1 0 0, limit lower=-3.14 upper=3.14 effort=30 velocity=0.6
- added joint left_joint4: type continuous, parent left_link3, child left_link4, origin xyz=-0.226 0.0 0.152 rpy=0 0 1.57, axis 0 0 1, limit lower=-3.14 upper=-0.9 effort=30 velocity=0.6
- added joint left_joint5: type revolute, parent left_link4, child left_link5, origin xyz=0 0.0 0.183 rpy=-3.14 0 1.57, axis 0 1 0, limit lower=-3.14 upper=-0.9 effort=30 velocity=0.6
- added joint left_joint6: type continuous, parent left_link5, child left_link6, origin xyz=0 0.0 0.005 rpy=0 0 3.14, axis 0 0 1, limit lower=-3.14 upper=3.14 effort=30 velocity=0.6
- added joint right_joint1: type continuous, parent base_link, child right_link1, origin xyz=0.19 0.2 0.206 rpy=0 0 -0.785, axis 0 0 1, limit lower=-3.14 upper=3.14 effort=30 velocity=0.6
- added joint right_joint2: type continuous, parent right_link1, child right_link2, origin xyz=0.2 0.0 0.446 rpy=1.57 0 0, axis 1 0 0, limit lower=-3.14 upper=3.14 effort=30 velocity=0.6
- added joint right_joint3: type continuous, parent right_link2, child right_link3, origin xyz=-0.08 0 0.41 rpy=3.14 0 0, axis 1 0 0, limit lower=-3.14 upper=3.14 effort=30 velocity=0.6
- added joint right_joint4: type continuous, parent right_link3, child right_link4, origin xyz=-0.226 0.0 0.152 rpy=0 0 1.57, axis 0 0 1, limit lower=-3.14 upper=-0.9 effort=30 velocity=0.6
- added joint right_joint5: type revolute, parent right_link4, child right_link5, origin xyz=0 0.0 0.183 rpy=-3.14 0 1.57, axis 0 1 0, limit lower=-3.14 upper=-0.9 effort=30 velocity=0.6
- added joint right_joint6: type continuous, parent right_link5, child right_link6, origin xyz=0 0.0 0.005 rpy=0 0 3.14, axis 0 0 1, limit lower=-3.14 upper=3.14 effort=30 velocity=0.6

Commit message: added controller files and programatic moveit code

File: mara.urdf (robot description, URDF)
Before this commit: robot mara, 13 links, 12 joints
Links:
- added link camera_base_link; visual box size=0.3 0.6 1.0
Joints:
- added joint camera_joint: type fixed, parent base_link, child camera_base_link, origin xyz=0 0 0 rpy=0 0 0, axis 0 0 0

Commit message: updated gripper position command functionality

File: mara.urdf (robot description, URDF)
Before this commit: robot mara, 14 links, 13 joints
Links:
- link base_link: geometry visual mesh filename=package://mara/models/MARA_wheeled_base.dae scale=0.001 0.001 0.001
Joints:
- joint left_joint1: origin xyz=-0.19 0.2 0.206 rpy=0 0 0.785 -> xyz=-0.165 0.2 0.206 rpy=0 0 0.785
- joint right_joint1: origin xyz=0.19 0.2 0.206 rpy=0 0 -0.785 -> xyz=0.165 0.2 0.206 rpy=0 0 -0.785

Commit message: added OPE and object retrieval to control script

File: mara.urdf (robot description, URDF)
Before this commit: robot mara, 14 links, 13 joints
Links:
- link camera_base_link: geometry visual box size=0.25 0.6 1.0
